Commit message: Prepare for simulation trials

File: src/khm2_description/urdf/khm2.urdf.xacro (robot description, xacro)
@@ -1,4 +1,5 @@
 <?xml version="1.0" encoding="utf-8"?>
-<robot name="khm2">
+<robot name="khm2" xmlns:xacro="http://www.ros.org/wiki/xacro">
+<xacro:include filename="$(find khm2_description)/urdf/macro.xacro"/>
 <link name="FL_wheel_link">
   <visual>
@@ -17,6 +18,6 @@
     <origin xyz="0 0 0"/>
     <inertia
-	    ixx="3" ixy="3" ixz="3"
-	    iyy="3" iyz="3" izz="3"/>
+	    ixx="0.003" ixy="0" ixz="0"
+	    iyy="0.003" iyz="0" izz="0.003"/>
   </inertial>
 </link>
@@ -37,6 +38,6 @@
     <origin xyz="0 0 0"/>
     <inertia
-	    ixx="3" ixy="3" ixz="3"
-	    iyy="3" iyz="3" izz="3"/>
+	    ixx="0.003" ixy="0" ixz="0"
+	    iyy="0.003" iyz="0" izz="0.003"/>
   </inertial>
 </link>
@@ -57,6 +58,6 @@
     <origin xyz="0 0 0"/>
     <inertia
-	    ixx="3" ixy="3" ixz="3"
-	    iyy="3" iyz="3" izz="3"/>
+	    ixx="0.003" ixy="0" ixz="0"
+	    iyy="0.003" iyz="0" izz="0.003"/>
   </inertial>
 </link>
@@ -77,6 +78,6 @@
     <origin xyz="0 0 0"/>
     <inertia
-	    ixx="3" ixy="3" ixz="3"
-	    iyy="3" iyz="3" izz="3"/>
+	    ixx="0.003" ixy="0" ixz="0"
+	    iyy="0.003" iyz="0" izz="0.003"/>
   </inertial>
 </link>
@@ -94,6 +95,6 @@
   </collision>
   <inertial>
-	  <mass value="30"/>
-          <inertia ixx="3" ixy="3" ixz="3" iyy="3" iyz="3" izz="3" />
+      <mass value="3.0"/>
+      <xacro:box_inertia m="3.0" x="0.333" y="0.16125" z="0.15428"/>
   </inertial>
 </link>

Commit message: Collision & Integration with TaRO

File: src/khm2_description/urdf/khm2.urdf.xacro (robot description, xacro)
@@ -6,18 +6,16 @@
     <origin rpy="0 0 0" xyz="0 0 0"/>
     <geometry>
-      <mesh filename="package://khm2_description/models/wheel.dae"/>
+      <mesh filename="package://khm2_description/models/wheel.stl"/>
     </geometry>
   </visual>
   <collision>
     <geometry>
-      <mesh filename="package://khm2_description/models/wheel.dae"/>
+      <mesh filename="package://khm2_description/models/wheel_col.dae"/>
     </geometry>
   </collision>
   <inertial>
-    <mass value="0.45"/>
+    <mass value="0.06925"/>
     <origin xyz="0 0 0"/>
-    <inertia
-	    ixx="0.003" ixy="0" ixz="0"
-	    iyy="0.003" iyz="0" izz="0.003"/>
+    <xacro:cylinder_inertia m="0.06925" r="0.112" h="0.127"/>
   </inertial>
 </link>
@@ -26,18 +24,16 @@
     <origin rpy="0 0 0" xyz="0 0 0"/>
     <geometry>
-      <mesh filename="package://khm2_description/models/wheel.dae"/>
+      <mesh filename="package://khm2_description/models/wheel.stl"/>
     </geometry>
   </visual>
   <collision>
     <geometry>
-      <mesh filename="package://khm2_description/models/wheel.dae"/>
+      <mesh filename="package://khm2_description/models/wheel_col.dae"/>
     </geometry>
   </collision>
   <inertial>
-    <mass value="0.45"/>
+    <mass value="0.06925"/>
     <origin xyz="0 0 0"/>
-    <inertia
-	    ixx="0.003" ixy="0" ixz="0"
-	    iyy="0.003" iyz="0" izz="0.003"/>
+    <xacro:cylinder_inertia m="0.06925" r="0.112" h="0.127"/>
   </inertial>
 </link>
@@ -46,18 +42,16 @@
     <origin rpy="0 0 0" xyz="0 0 0"/>
     <geometry>
-      <mesh filename="package://khm2_description/models/wheel.dae"/>
+      <mesh filename="package://khm2_description/models/wheel.stl"/>
     </geometry>
   </visual>
   <collision>
     <geometry>
-      <mesh filename="package://khm2_description/models/wheel.dae"/>
+      <mesh filename="package://khm2_description/models/wheel_col.dae"/>
     </geometry>
   </collision>
   <inertial>
-    <mass value="0.45"/>
+    <mass value="0.06925"/>
     <origin xyz="0 0 0"/>
-    <inertia
-	    ixx="0.003" ixy="0" ixz="0"
-	    iyy="0.003" iyz="0" izz="0.003"/>
+    <xacro:cylinder_inertia m="0.06925" r="0.112" h="0.127"/>
   </inertial>
 </link>
@@ -66,18 +60,16 @@
     <origin rpy="0 0 0" xyz="0 0 0"/>
     <geometry>
-      <mesh filename="package://khm2_description/models/wheel.dae"/>
+      <mesh filename="package://khm2_description/models/wheel.stl"/>
     </geometry>
   </visual>
   <collision>
     <geometry>
-      <mesh filename="package://khm2_description/models/wheel.dae"/>
+      <mesh filename="package://khm2_description/models/wheel_col.dae"/>
     </geometry>
   </collision>
   <inertial>
-    <mass value="0.45"/>
+    <mass value="0.06925"/>
     <origin xyz="0 0 0"/>
-    <inertia
-	    ixx="0.003" ixy="0" ixz="0"
-	    iyy="0.003" iyz="0" izz="0.003"/>
+    <xacro:cylinder_inertia m="0.06925" r="0.112" h="0.127"/>
   </inertial>
 </link>
@@ -95,6 +87,6 @@
   </collision>
   <inertial>
-      <mass value="3.0"/>
-      <xacro:box_inertia m="3.0" x="0.333" y="0.16125" z="0.15428"/>
+      <mass value="2.0"/>
+      <xacro:box_inertia m="2.0" x="0.333" y="0.16125" z="0.15428"/>
   </inertial>
 </link>
@@ -126,4 +118,14 @@
 <gazebo>
    <plugin filename="libgazebo_ros_control.so" name="gazebo_ros_control"></plugin>
+   <plugin name="p3d_base_controller" filename="libgazebo_ros_p3d.so">
+    <alwaysOn>true</alwaysOn>
+    <updateRate>50.0</updateRate>
+    <bodyName>base_link</bodyName>
+    <topicName>odom</topicName>
+    <gaussianNoise>0</gaussianNoise>
+    <frameName>world</frameName>
+    <xyzOffsets>0 0 0</xyzOffsets>
+    <rpyOffsets>0 0 0</rpyOffsets>
+  </plugin>
 </gazebo>
   <transmission name="FR_trans">

Commit message: changes

File: src/khm2_description/urdf/khm2.urdf.xacro (robot description, xacro)
@@ -6,10 +6,10 @@
     <origin rpy="0 0 0" xyz="0 0 0"/>
     <geometry>
-      <mesh filename="package://khm2_description/models/wheel.stl"/>
+      <mesh filename="package://khm2_description/models/smooth.stl"/>
     </geometry>
   </visual>
   <collision>
     <geometry>
-      <mesh filename="package://khm2_description/models/wheel_col.dae"/>
+      <mesh filename="package://khm2_description/models/smooth_col.dae"/>
     </geometry>
   </collision>
@@ -24,10 +24,10 @@
     <origin rpy="0 0 0" xyz="0 0 0"/>
     <geometry>
-      <mesh filename="package://khm2_description/models/wheel.stl"/>
+      <mesh filename="package://khm2_description/models/smooth.stl"/>
     </geometry>
   </visual>
   <collision>
     <geometry>
-      <mesh filename="package://khm2_description/models/wheel_col.dae"/>
+      <mesh filename="package://khm2_description/models/smooth_col.dae"/>
     </geometry>
   </collision>
@@ -42,10 +42,10 @@
     <origin rpy="0 0 0" xyz="0 0 0"/>
     <geometry>
-      <mesh filename="package://khm2_description/models/wheel.stl"/>
+      <mesh filename="package://khm2_description/models/smooth.stl"/>
     </geometry>
   </visual>
   <collision>
     <geometry>
-      <mesh filename="package://khm2_description/models/wheel_col.dae"/>
+      <mesh filename="package://khm2_description/models/smooth_col.dae"/>
     </geometry>
   </collision>
@@ -60,10 +60,10 @@
     <origin rpy="0 0 0" xyz="0 0 0"/>
     <geometry>
-      <mesh filename="package://khm2_description/models/wheel.stl"/>
+      <mesh filename="package://khm2_description/models/smooth.stl"/>
     </geometry>
   </visual>
   <collision>
     <geometry>
-      <mesh filename="package://khm2_description/models/wheel_col.dae"/>
+      <mesh filename="package://khm2_description/models/smooth_col.dae"/>
     </geometry>
   </collision>

Commit message: Aaaah

File: src/khm2_description/urdf/khm2.urdf.xacro (robot description, xacro)
@@ -112,5 +112,4 @@
 	<hardwareInterface>hardware_interface/VelocityJointInterface</hardwareInterface>
 	<origin xyz="0.145 -0.145225 -0.1" rpy="0 0 0"/>
-	<origin xyz="-0.145 -0.145225 -0.1" rpy="0 0 0"/>
 	<child link="BR_wheel_link"/>
 	<parent link="base_link"/>

Commit message: fixed rover rotation

File: src/khm2_description/urdf/khm2.urdf.xacro (robot description, xacro)
@@ -93,5 +93,5 @@
 <joint name="FL_TO_BASELINK" type="continuous">
 	<hardwareInterface>hardware_interface/VelocityJointInterface</hardwareInterface>
-	<origin xyz="-0.145 0.145225 -0.1" rpy="0 0 0"/>
+	<origin xyz="0.145225 0.145 -0.1" rpy="0 0 1.5707"/>
 	<child link="FL_wheel_link"/>
 	<parent link="base_link"/>
@@ -99,5 +99,5 @@
 <joint name="FR_TO_BASELINK" type="continuous">
 	<hardwareInterface>hardware_interface/VelocityJointInterface</hardwareInterface>
-	<origin xyz="0.145 0.145225 -0.1" rpy="0 0 0"/>
+	<origin xyz="0.145225 -0.145 -0.1" rpy="0 0 1.5707"/>
 	<child link="FR_wheel_link"/>
 	<parent link="base_link"/>
@@ -105,5 +105,5 @@
 <joint name="BL_TO_BASELINK" type="continuous">
 	<hardwareInterface>hardware_interface/VelocityJointInterface</hardwareInterface>
-	<origin xyz="-0.145 -0.145225 -0.1" rpy="0 0 0"/>
+	<origin xyz="-0.14225 0.145 -0.1" rpy="0 0 1.5707"/>
 	<child link="BL_wheel_link"/>
 	<parent link="base_link"/>
@@ -111,6 +111,5 @@
 <joint name="BR_TO_BASELINK" type="continuous">
 	<hardwareInterface>hardware_interface/VelocityJointInterface</hardwareInterface>
-	<origin xyz="0.145 -0.145225 -0.1" rpy="0 0 0"/>
-	<origin xyz="-0.145 -0.145225 -0.1" rpy="0 0 0"/>
+	<origin xyz="-0.145225 -0.145 -0.1" rpy="0 0 1.5707"/>
 	<child link="BR_wheel_link"/>
 	<parent link="base_link"/>

Commit message: hi bret

File: src/khm2_description/urdf/khm2.urdf.xacro (robot description, xacro)
@@ -87,5 +87,5 @@
   </collision>
   <inertial>
-      <mass value="2.0"/>
+      <mass value="2.3"/>
       <xacro:box_inertia m="2.0" x="0.333" y="0.16125" z="0.15428"/>
   </inertial>
@@ -93,9 +93,5 @@
 <joint name="FL_TO_BASELINK" type="continuous">
 	<hardwareInterface>hardware_interface/VelocityJointInterface</hardwareInterface>
-<<<<<<< HEAD
-	<origin xyz="-0.145 0.145225 -0.1" rpy="0 0 0"/>
-=======
 	<origin xyz="0.145225 0.145 -0.1" rpy="0 0 1.5707"/>
->>>>>>> d6e6974418bc85c990dd74811f846e600c1a50ca
 	<child link="FL_wheel_link"/>
 	<parent link="base_link"/>
@@ -103,9 +99,5 @@
 <joint name="FR_TO_BASELINK" type="continuous">
 	<hardwareInterface>hardware_interface/VelocityJointInterface</hardwareInterface>
-<<<<<<< HEAD
-	<origin xyz="0.145 0.145225 -0.1" rpy="0 0 0"/>
-=======
 	<origin xyz="0.145225 -0.145 -0.1" rpy="0 0 1.5707"/>
->>>>>>> d6e6974418bc85c990dd74811f846e600c1a50ca
 	<child link="FR_wheel_link"/>
 	<parent link="base_link"/>
@@ -113,9 +105,5 @@
 <joint name="BL_TO_BASELINK" type="continuous">
 	<hardwareInterface>hardware_interface/VelocityJointInterface</hardwareInterface>
-<<<<<<< HEAD
-	<origin xyz="-0.145 -0.145225 -0.1" rpy="0 0 0"/>
-=======
 	<origin xyz="-0.14225 0.145 -0.1" rpy="0 0 1.5707"/>
->>>>>>> d6e6974418bc85c990dd74811f846e600c1a50ca
 	<child link="BL_wheel_link"/>
 	<parent link="base_link"/>
@@ -123,6 +111,5 @@
 <joint name="BR_TO_BASELINK" type="continuous">
 	<hardwareInterface>hardware_interface/VelocityJointInterface</hardwareInterface>
-<<<<<<< HEAD
-	<origin xyz="0.145 -0.145225 -0.1" rpy="0 0 0"/>
+	<origin xyz="-0.145 -0.145225 -0.1" rpy="0 0 1.5707"/>
 	<child link="BR_wheel_link"/>
 	<parent link="base_link"/>
